File: ledPCBFiles/ledPCBFiles.kicad_sch (KiCad schematic)
At the start: 14 parts, among them U1 LM555xN, U2 74LS161

Commit message: Edit capacitor value
Parts:
- C1: value 100n -> 10n
Changed lines of the file:
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@@
 			)
 		)
-		(property "Value" "100n"
+		(property "Value" "10n"
 			(at 102.87 59.6835 0)
 			(show_name no)
